File: Microcontroller.sch (KiCad schematic (older format))
At the start: 0 parts

Commit message: Added temp circuit for current sense
Parts:
- added C? (x8): 0.1u, Capacitor_SMD:C_0603_1608Metric, symbol Device:C_Small
- added U?: STM32F302C6Tx, Package_QFP:LQFP-48_7x7mm_P0.5mm, symbol MCU_ST_STM32F3:STM32F302C6Tx
Connections:
- new net +3.3VA: U?.9 (VDDA)
- new net +3V3: C?.1, C?.1, C?.1, C?.1, C?.1, C?.1, C?.1, C?.1, U?.1 (VBAT), U?.24 (VDD), U?.36 (VDD), U?.48 (VDD)
- new net GND: C?.2, C?.2, C?.2, C?.2, C?.2, C?.2, C?.2, C?.2, U?.23 (VSS), U?.35 (VSS), U?.47 (VSS)
- new net GNDA: U?.8 (VSSA)
Other:
- note added: "Microcontroller Decoupling"
