File: Microcontroller.sch (KiCad schematic (older format))
At the start: 35 parts, among them J201 Conn_02x05_Odd_Even, SW201 B3U-1100P, U201 STM32F302C6Tx, U202 NCV7357, X201 OSC_4PIN

Commit message: Initial routing complete
Connections:
- net SWCLK is gone; now on net SWDCLK: U201.37 (PA14)
Changed lines of the file:
@@
 TRACESWO
 Text Label 10850 5550 2    50   ~ 0
-SWCLK
+SWDCLK
 Text Label 10850 5450 2    50   ~ 0
 SWDIO
@@
 Wire Wire Line
 	9400 2700 9400 2850
-Wire Bus Line
-	10400 4650 10400 5150
-Wire Bus Line
-	4750 2200 4750 4450
 Connection ~ 9300 2700
 $Comp
@@
 	1    0    0    -1
 $EndComp
+Wire Bus Line
+	10400 4650 10400 5150
+Wire Bus Line
+	4750 2200 4750 4450
 $EndSCHEMATC

Commit message: Minor updates
Connections:
- net CANH is gone; now on net CAN+: R203.1
- net CANL is gone; now on net CAN-: R208.2
Changed lines of the file:
@@
 	4100 6250 2900 6250
 Text HLabel 3300 6150 0    50   BiDi ~ 0
-CANL
+CAN-
 Text HLabel 3300 4950 0    50   BiDi ~ 0
-CANH
+CAN+
 $Comp
 L power:GND #PWR0215
