File: Communication.sch (KiCad schematic (older format))
At the start: 0 parts

Commit message: Added USB Connector
Parts:
- added F?: 1A, symbol Device:Fuse_Small
- added FB?: FerriteBead_Small, symbol Device:FerriteBead_Small
- added J?: USB_C_Receptacle_USB2.0, symbol Connector:USB_C_Receptacle_USB2.0
- added L?: L_Coupled_Small_1324, symbol Device:L_Coupled_Small_1324
- added R? (x2): 5k, symbol Device:R_Small
- added U? (x2): TPD1E05U06PYR, symbol ReflowOven:TPD1E05U06PYR
Connections:
- new net: F?.1, J?.A4 (VBUS), J?.A9 (VBUS), J?.B4 (VBUS), J?.B9 (VBUS)
- new net: J?.A5 (CC1), R?.2
- new net: J?.A6 (D+), J?.B6 (D+), L?.2
- new net: J?.A7 (D-), J?.B7 (D-), L?.1
- new net: J?.B5 (CC2), R?.1
- new net: FB?.2, J?.S1 (SHIELD)
- new net +5V: F?.2
- new net GND: FB?.1, J?.A1 (GND), J?.A12 (GND), J?.B1 (GND), J?.B12 (GND), R?.1, R?.2, U?.2 (GND), U?.2 (GND)
- new net USB_DM: L?.3, U?.1 (PROT)
- new net USB_DP: L?.4, U?.1 (PROT)
- no-connect marks 0 -> 2
Other:
- note added: "USB Connection"
