File: ThermocoupleAmp.sch (KiCad schematic (older format))
At the start: 0 parts

Commit message: Added display driver for 7 segment
Parts:
- added C?: 0.1u, symbol Device:C_Small
- added C?: 10uF, symbol Device:C_Small
- added J?: Conn_01x02_Male, symbol Connector:Conn_01x02_Male
- added R?: 1M, symbol Device:R_Small
- added R? (x2): 2M, symbol Device:R_Small
- added U?: MCP96RL01T, symbol ReflowOven:MCP96RL01T
Connections:
- new net: J?.2 (Pin_2), U?.2 (Vin+)
- new net: J?.1 (Pin_1), R?.1, U?.4 (Vin-)
- new net: R?.2, R?.2, U?.6 (V_Sense)
- new net +3.3VA: C?.1, C?.2, R?.1, U?.8 (VDD)
- new net GNDA: C?.1, C?.2, R?.1, R?.2, U?.1 (GND), U?.10 (GND), U?.13 (GND), U?.16 (ADDR), U?.17 (GND), U?.18 (GND), U?.3 (GND), U?.5 (GND)
- new net I2C_SCL: U?.19 (SCL)
- new net I2C_SDA: U?.20 (SDA)
- no-connect marks 0 -> 6
Other:
- note added: "I2C Address = 1100 000 = 0xC0"
