File: ThermocoupleAmp.sch (KiCad schematic (older format))
At the start: 7 parts, among them J601 Thermocouple_Conn, U601 MCP96RL01T

Commit message: Done with footprints
Parts:
- J601: footprint (none) -> ReflowOven:PRT-13612
Changed lines of the file:
@@
 F 0 "J601" H 7272 3832 50  0000 R CNN
 F 1 "Thermocouple_Conn" H 7272 3923 50  0000 R CNN
-F 2 "" H 7300 3950 50  0001 C CNN
+F 2 "ReflowOven:PRT-13612" H 7300 3950 50  0001 C CNN
 F 3 "~" H 7300 3950 50  0001 C CNN
 	1    7300 3950
