File: ReflowOven.kicad_pcb (KiCad board)
At the start: 4 copper layers, 145 parts, among them J201 Conn_02x05_Counter_Clockwise, J401 SD_Card, J501 IEC320-C14, J502 IEC-NEMA-3PIN, J601 Thermocouple_Conn, J701 Conn_01x03_Male, J702 Microfit-4pin, J703 Conn_01x06_Male, J704 USB_C_Receptacle_USB2.0, K501 G5RLU1E, P501 RAC10-3.3SK_277, SW201 B3U-1100P, SW401 SW_Push, SW402 SW_Push, SW403 SW_Push, SW404 RotaryEncoder_Switch, U201 STM32F302C6Tx, U202 NCV7357, U301 PCF5331ATT_AJ, U401 74HC193, U402 TCA9534, U403 74HC193, U404 HEF4013B, U405 SN74LVC2G08, U406 74LVC2G14, U407 74HC86D, U408 HEF4013B, U501 MAX4684_5, U502 INA226, U601 MCP96RL01T, U701 TPD1E05U06PYR, U702 TPD1E05U06PYR, X201 OSC_4PIN, X401 OSC_4PIN

Commit message: Began routing
Parts:
- removed F701: 1A, ReflowOven:FUSC6125X279N
- removed FB401: FerriteBead_Small, Inductor_SMD:L_0603_1608Metric
- removed J401: SD_Card, ReflowOven:AMPHENOL-10067847
- added REF**: MountingHole_3.2mm_M3_Pad_Via, MountingHole:MountingHole_3.2mm_M3_Pad_Via, F.Cu at (120.9, 92.2)
- added REF**: MountingHole_3.2mm_M3_Pad_Via, MountingHole:MountingHole_3.2mm_M3_Pad_Via, F.Cu at (23.4, 31.8)
- added REF**: MountingHole_3.2mm_M3_Pad_Via, MountingHole:MountingHole_3.2mm_M3_Pad_Via, F.Cu at (23.4, 106.4)
- added REF**: MountingHole_3.2mm_M3_Pad_Via, MountingHole:MountingHole_3.2mm_M3_Pad_Via, F.Cu at (24.4, 175.0)
- added REF**: MountingHole_3.2mm_M3_Pad_Via, MountingHole:MountingHole_3.2mm_M3_Pad_Via, F.Cu at (168.8, 174.5)
- added REF**: MountingHole_3.2mm_M3_Pad_Via, MountingHole:MountingHole_3.2mm_M3_Pad_Via, F.Cu at (168.7, 31.8)
- added REF**: MountingHole_3.2mm_M3_Pad_Via, MountingHole:MountingHole_3.2mm_M3_Pad_Via, F.Cu at (120.9, 31.8)
- added REF**: MountingHole_3.2mm_M3_Pad_Via, MountingHole:MountingHole_3.2mm_M3_Pad_Via, F.Cu at (23.4, 92.2)
- added REF**: MountingHole_3.2mm_M3_Pad_Via, MountingHole:MountingHole_3.2mm_M3_Pad_Via, F.Cu at (106.7, 92.2)
- added REF**: MountingHole_3.2mm_M3_Pad_Via, MountingHole:MountingHole_3.2mm_M3_Pad_Via, F.Cu at (106.7, 31.8)
- added U409: SD-Card-NOSHELL, ReflowOven:AMPHENOL-10067847, F.Cu at (144.5, 91.9)
- moved R305 148.8 mm to (52.8, 65.8)
- moved J501 138.4 mm to (56.4, 169.4), turned to 270 degrees
- moved R313 131.9 mm to (69.6, 61.2), turned to 180 degrees
- moved SW401 125.4 mm to (30.4, 43.3), turned to 90 degrees
- moved R303 123.7 mm to (52.8, 62.7)
- moved R302 119.9 mm to (52.8, 61.2)
- moved R306 119.7 mm to (52.8, 67.3)
- moved C408 117.3 mm to (38.8, 55.1)
- moved C302 116.7 mm to (55.9, 61.2), turned to 270 degrees
- moved R304 116.1 mm to (52.8, 64.3)
- moved R307 115.9 mm to (52.8, 68.8)
- moved C301 113.2 mm to (55.9, 58.2), turned to 90 degrees
- moved R301 113.0 mm to (52.8, 59.7)
- moved R308 110.9 mm to (69.6, 68.8), turned to 180 degrees
- moved C409 107.3 mm to (38.6, 61.7)
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Connections:
- net /Communication/USB_DM renamed /Communication/USB_D-
- net /Communication/USB_DP renamed /Communication/USB_D+
- F502 pad 1: /MainsPower/VACL -> Net-(F502-Pad1)
- F502 pad 2: Net-(F502-Pad2) -> /MainsPower/VACL
- K501 pad 3: Net-(F502-Pad2) -> Net-(F502-Pad1)
- K501 pad 6: Net-(F502-Pad2) -> Net-(F502-Pad1)
- U201 pad 42: Net-(U201-Pad42) -> /HumanInterface/SW_BTN
- U201 pad 9: +3.3VA -> +3V3
- U401 pad 1: (no net) -> GND
- U401 pad 10: (no net) -> GND
- U401 pad 13: (no net) -> Net-(U401-Pad13)
- U401 pad 9: (no net) -> GND
- U403 pad 1: (no net) -> GND
- U403 pad 10: (no net) -> GND
- U403 pad 13: (no net) -> Net-(U403-Pad13)
- U403 pad 4: Net-(U401-Pad~) -> Net-(U401-Pad13)
- U403 pad 9: (no net) -> GND
Routing:
- net /Microcontroller/DLED0: track 0.00 -> 72.2 mm
- net /Microcontroller/DLED1: track 0.00 -> 71.5 mm
- net /Microcontroller/DLED2: track 0.00 -> 70.8 mm
- net /Microcontroller/DLED3: track 0.00 -> 69.6 mm
- net GND: track 0.00 -> 69.5 mm, vias 0 -> 38
- net /Communication/USB_D+: track 0.00 -> 42.6 mm
- net /Communication/USB_D-: track 0.00 -> 41.7 mm
- net +3V3: track 0.00 -> 41.2 mm, vias 0 -> 19
- net /Display/I2C_SCL: track 0.00 -> 39.5 mm
- net /Display/I2C_SDA: track 0.00 -> 39.3 mm
- net /Microcontroller/DLED4: track 0.00 -> 39.0 mm
- net Net-(D205-Pad1): track 0.00 -> 23.0 mm
- net Net-(D204-Pad1): track 0.00 -> 23.0 mm
- net Net-(D203-Pad1): track 0.00 -> 22.9 mm
- net Net-(D206-Pad1): track 0.00 -> 22.9 mm
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- added copper zone on F.Cu, net +3.3VA
- added copper zone on In2.Cu, net +3V3
- added copper zone on F.Cu, net GND
- added copper zone on In1.Cu, net GND
- added copper zone on F.Cu, net Net-(FB701-Pad2)
Other:
- board outline added: 157.5 x 155.4 mm
- rule trace_min: 0.2 -> 0.127
- board text added: "3.3V Power"

Commit message: Continuing routes
Parts:
- moved C207 4.46 mm to (106.4, 131.4)
- moved C212 4.14 mm to (124.5, 134.1)
- moved C206 3.69 mm to (132.7, 131.4)
- moved C403 2.57 mm to (75.1, 88.3), turned to 0 degrees
- moved R309 0.89 mm to (70.5, 67.4), turned to 180 degrees
- moved R308 0.89 mm to (70.5, 68.8)
- moved R310 0.89 mm to (70.5, 65.8)
- moved R311 0.89 mm to (70.5, 64.3)
- moved R312 0.89 mm to (70.5, 62.7)
- moved R313 0.89 mm to (70.5, 61.2)
- moved R314 0.89 mm to (70.5, 59.7)
- moved R315 0.89 mm to (70.5, 58.2)
- moved R316 0.89 mm to (70.5, 56.6)
- moved C407 0.61 mm to (89.5, 55.7)
- moved C415 0.57 mm to (100.3, 69.8)
Routing:
- net /Display/SEG7: track 0.00 -> 108.3 mm, vias 0 -> 2
- net /Display/SEG13: track 0.00 -> 95.4 mm
- net /HumanInterface/SW3: track 0.00 -> 94.7 mm, vias 0 -> 1
- net /Display/SEG10: track 0.00 -> 86.7 mm
- net GND: track 69.5 -> 154.5 mm, vias 38 -> 84
- net /Display/SEG14: track 0.00 -> 80.4 mm
- net /HumanInterface/SW2: track 0.00 -> 79.3 mm, vias 0 -> 1
- net /HumanInterface/SW1: track 0.00 -> 78.5 mm, vias 0 -> 1
- net /Microcontroller/DLED5: track 0.00 -> 77.2 mm, vias 0 -> 2
- net /HumanInterface/SW_BTN: track 1.40 -> 72.7 mm
- net /Display/SEG4: track 0.00 -> 59.2 mm, vias 0 -> 2
- net /Display/SEG2: track 0.00 -> 58.9 mm
- net /Display/SEG12: track 0.00 -> 58.4 mm
- net /Display/SEG6: track 0.00 -> 54.2 mm
- net /Display/SEG11: track 0.00 -> 53.5 mm
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- added copper zone on F.Cu, net +3V3
- added copper zone on B.Cu, net /Display/COM0
- added copper zone on F.Cu, net /Display/COM0
- added copper zone on B.Cu, net /Display/COM1
- added copper zone on F.Cu, net /Display/COM1

Commit message: Footprint update
Parts:
- J201: value Conn_02x05_Counter_Clockwise -> Conn_02x05_Odd_Even
- moved J201 0.13 mm to (151.8, 78.2)
Connections:
- J201 pad 10: /Microcontroller/SWDIO -> /Microcontroller/~RST
- J201 pad 2: GND -> /Microcontroller/SWDIO
- J201 pad 4: Net-(J201-Pad4) -> /Microcontroller/SWDCLK
- J201 pad 6: /Microcontroller/~RST -> /Microcontroller/TRACESWO
- J201 pad 8: /Microcontroller/TRACESWO -> Net-(J201-Pad8)
- J201 pad 9: /Microcontroller/SWDCLK -> GND
Routing:
- net GND: track 154.5 -> 162.9 mm, vias 84 -> 87

Commit message: Done for today with layout
Parts:
- moved P501 13.2 mm to (46.1, 142.2)
- moved F501 9.08 mm to (58.0, 166.2), turned to 0 degrees
- moved F502 5.72 mm to (73.2, 175.1)
- moved J501 5.72 mm to (56.4, 175.1)
- moved C506 1.02 mm to (70.1, 122.7)
- moved C507 1.02 mm to (70.1, 121.2)
- moved R502 1.02 mm to (67.1, 122.7)
Connections:
- J702 pad 2: /Communication/CANL -> /Communication/CAN-
- J702 pad 3: /Communication/CANH -> /Communication/CAN+
- R203 pad 1: /Communication/CANH -> /Microcontroller/CANH
- R208 pad 2: /Communication/CANL -> /Microcontroller/CANL
- U202 pad 6: /Communication/CANL -> /Communication/CAN-
- U202 pad 7: /Communication/CANH -> /Communication/CAN+
Routing:
- net /Communication/UART_RTS: track 2.90 -> 118.6 mm
- net /Communication/UART_TX: track 2.67 -> 116.1 mm
- net /Communication/UART_RX: track 1.89 -> 114.9 mm
- net /Communication/UART_CTS: track 4.30 -> 116.9 mm
- net /MainsPower/VACN: track 0.00 -> 97.9 mm, vias 0 -> 2
- net GNDPWR: track 0.00 -> 91.4 mm
- net /Communication/CAN+: track 0.00 -> 69.4 mm, vias 0 -> 1
- net /Communication/CAN-: track 0.00 -> 68.4 mm, vias 0 -> 1
- net Net-(F502-Pad1): track 0.00 -> 53.4 mm
- net /MainsPower/RELAY_SET: track 2.13 -> 42.4 mm
- net Net-(K501-Pad1): track 0.00 -> 37.8 mm, vias 0 -> 1
- net Net-(K501-Pad8): track 0.00 -> 36.0 mm, vias 0 -> 1
- net /MainsPower/CURRENT_ALRT: track 2.68 -> 31.6 mm, vias 1 -> 2
- net /MainsPower/LN_OUT: track 0.00 -> 22.6 mm
- net GND: track 162.9 -> 183.6 mm, vias 87 -> 98
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- added copper zone on F.Cu, net /MainsPower/3V3_REG_OUT
- added copper zone on F.Cu, net /MainsPower/VACL
- added copper zone on F.Cu, net Net-(F502-Pad1)

Commit message: Initial routing complete
Parts:
- added REF**: PinHeader_1x10_P1.00mm_Vertical, Connector_PinHeader_1.00mm:PinHeader_1x10_P1.00mm_Vertical, F.Cu at (78.4, 103.6)
- added REF**: PinHeader_1x10_P1.00mm_Vertical, Connector_PinHeader_1.00mm:PinHeader_1x10_P1.00mm_Vertical, F.Cu at (78.4, 94.4)
- added REF**: PinHeader_1x10_P1.00mm_Vertical, Connector_PinHeader_1.00mm:PinHeader_1x10_P1.00mm_Vertical, F.Cu at (78.4, 99.3)
- moved C510 10.00 mm to (76.2, 117.3), turned to 90 degrees
- moved C511 7.97 mm to (77.7, 117.3), turned to 90 degrees
- moved C512 6.04 mm to (79.2, 117.3), turned to 90 degrees
- moved C516 4.58 mm to (85.3, 117.3), turned to 90 degrees
- moved C513 4.32 mm to (80.8, 117.3), turned to 90 degrees
- moved C515 3.30 mm to (83.8, 117.3), turned to 90 degrees
- moved C514 3.18 mm to (82.3, 117.3), turned to 90 degrees
- moved C402 2.05 mm to (142.6, 101.1), turned to 90 degrees
Connections:
- U201 pad 37: /Microcontroller/SWCLK -> /Microcontroller/SWDCLK
Routing:
- net /Display/I2C_SDA: track 86.5 -> 260.1 mm, vias 2 -> 5
- net /Display/I2C_SCL: track 86.2 -> 258.4 mm, vias 2 -> 5
- net /Microcontroller/~RST: track 12.0 -> 93.9 mm, vias 0 -> 1
- net /HumanInterface/SW2: track 84.5 -> 160.4 mm
- net /HumanInterface/SW3: track 101.1 -> 175.8 mm
- net /Microcontroller/TRACESWO: track 2.44 -> 75.4 mm
- net /Microcontroller/SWDIO: track 1.66 -> 74.3 mm
- net /HumanInterface/SW1: track 82.7 -> 154.0 mm
- net /Microcontroller/SWDCLK: track 0.00 -> 70.6 mm, vias 0 -> 1
- net /HumanInterface/SW_BTN: track 82.5 -> 137.3 mm
- net /HumanInterface/SPI_NSS: track 6.86 -> 55.3 mm, vias 1 -> 2
- net /HumanInterface/SD_DET: track 10.8 -> 57.7 mm, vias 1 -> 2
- net /HumanInterface/SPI_MOSI: track 7.43 -> 51.0 mm, vias 1 -> 2
- net /HumanInterface/SPI_SCK: track 7.08 -> 43.7 mm, vias 1 -> 2
- net /MainsPower/RELAY_SET: track 42.4 -> 76.3 mm, vias 1 -> 2
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- added copper zone on B.Cu, net +3V3

Commit message: Minor updates
Parts:
- J701: footprint Connector_PinHeader_1.00mm:PinHeader_1x03_P1.00mm_Vertical -> Connector_PinHeader_2.54mm:PinHeader_1x03_P2.54mm_Vertical
- J702: footprint Connector_PinHeader_1.00mm:PinHeader_2x02_P1.00mm_Vertical -> Connector_PinHeader_2.54mm:PinHeader_2x02_P2.54mm_Vertical
- J703: footprint Connector_PinHeader_1.00mm:PinHeader_1x06_P1.00mm_Vertical -> Connector_PinHeader_2.54mm:PinHeader_1x06_P2.54mm_Vertical
- moved J702 7.83 mm to (161.0, 67.0), turned to 270 degrees
- moved R205 7.58 mm to (161.7, 61.8)
- moved R208 7.58 mm to (160.9, 64.1)
- moved C203 7.58 mm to (158.4, 61.8)
- moved R203 7.58 mm to (162.2, 64.1)
- moved R206 7.58 mm to (158.4, 63.8)
- moved J701 5.17 mm to (167.8, 75.7), turned to 90 degrees
- moved J703 0.61 mm to (160.3, 79.8)
Connections:
- R203 pad 1: /Microcontroller/CANH -> /Communication/CAN+
- R208 pad 2: /Microcontroller/CANL -> /Communication/CAN-
- U409 pad GND: (no net) -> GND
Routing:
- net /Communication/CAN+: track 69.4 -> 85.5 mm
- net /Communication/CAN-: track 68.3 -> 76.8 mm
- net /Communication/UART_TX: track 116.1 -> 122.2 mm
- net GND: track 217.0 -> 222.5 mm, vias 103 -> 113
- net +3V3: track 127.9 -> 123.9 mm, vias 77 -> 76
- net /Communication/CANL: track 4.02 -> 0.00 mm
- net /Communication/UART_RX: track 114.9 -> 118.2 mm
- net /Communication/CANH: track 3.23 -> 0.00 mm
- net /Communication/UART_RTS: track 118.6 -> 120.4 mm
- net /MainsPower/VACN: track 97.9 -> 96.8 mm
- net /Communication/UART_CTS: track 116.9 -> 117.8 mm
Other:
- outline, holes or cut-outs redrawn
- net class Default: clearance 0.2 -> 0.125; trace_width 0.25 -> 0.127
- rule trace_clearance: 0.2 -> 0.125
- board text added: "3.3V"
- board text added: "CANH"
- board text added: "CANL"
- board text added: "CTS"
- board text added: "EARTH"
- board text added: "FTDI"
- board text added: "GND"
- board text added: "LIVE (L) / HOT"
- board text added: "NEUTRAL (N)"
- board text added: "PWR"
- board text added: "RTS"
- board text added: "RX"
- board text added: "SWD"
- board text added: "TERM JUMPERS"
- board text added: "TX"

Commit message: Added new model. Fixed board edge
Other:
- outline, holes or cut-outs redrawn
